File: pcb/headstage-interface.kicad_sch (KiCad schematic)
At the start: 4 parts, among them J1 DF40C(2.0)-70DS-0.4V(51), J5 DF40C(2.0)-70DS-0.4V(51)

Commit message: Added OEPS DESC.
Parts:
- J1, J5: OEPS DESC (none) -> CONNECTOR: CONN RCPT 70POS GOLD (OEPS D13 001) [DF40C(2.0)-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
- R4, R5: OEPS DESC (none) -> RESISTOR: SMD 0603 0Ω 1A [RCS06030000Z0EA ] [SMD]
Changed lines of the file:
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@@
 				)
 				(justify right)
+				(hide yes)
 			)
 		)
@@
 		)
 		(property "OEPSPN" "OEPS070090"
+			(at 198.12 83.82 0)
+			(effects
+				(font
+					(size 1.27 1.27)
+				)
+				(hide yes)
+			)
+		)
+		(property "OEPS DESC" "CONNECTOR:   CONN RCPT 70POS GOLD (OEPS D13 001)   [DF40C(2.0)-70DS-0.4V(51)] [SMD]"
 			(at 198.12 83.82 0)
 			(effects
@@
 			)
 		)
+		(property "OEPS DESC" "RESISTOR:   SMD 0603 0Ω 1A   [RCS06030000Z0EA ] [SMD]"
+			(at 195.58 147.32 0)
+			(effects
+				(font
+					(size 1.27 1.27)
+				)
+				(hide yes)
+			)
+		)
 		(pin "2"
 		)
@@
 				)
 				(justify right)
+				(hide yes)
 			)
 		)
@@
 		)
 		(property "OEPSPN" "OEPS070090"
+			(at 93.98 83.82 0)
+			(effects
+				(font
+					(size 1.27 1.27)
+				)
+				(hide yes)
+			)
+		)
+		(property "OEPS DESC" "CONNECTOR:   CONN RCPT 70POS GOLD (OEPS D13 001)   [DF40C(2.0)-70DS-0.4V(51)] [SMD]"
 			(at 93.98 83.82 0)
 			(effects
@@
 			(at 78.74 144.78 0)
 			(effects
+				(font
+					(size 1.27 1.27)
+				)
+				(hide yes)
+			)
+		)
+		(property "OEPS DESC" "RESISTOR:   SMD 0603 0Ω 1A   [RCS06030000Z0EA ] [SMD]"
+			(at 78.74 144.78 0)
+			(effects
