File: pcb/test-signal-interface.kicad_sch (KiCad schematic)
At the start: 7 parts, among them J2 BSE-040-01-F-D-A-TR, J3 BSE-040-01-F-D-A-TR, U1 AT24C64D-SSHM-T

Commit message: Added OEPS DESC.
Parts:
- C1: OEPS DESC (none) -> CAPACITOR: SMD CER 0402 100nF 25V ±10% X7R (OEPS H02 001) [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
- J2, J3: MPN BSE-040-01-X-D-A -> BSE-040-01-F-D-A-TR; OEPS DESC (none) -> CONNECTOR: CONN RCPT 80POS SMD GOLD [BSE-040-01-F-D-A-TR] [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
- R1, R2, R3: OEPS DESC (none) -> RESISTOR: SMD 0402 1kΩ ±1% 0.063W [CRCW04021K00FKED] [SMD]
- U1: OEPS DESC (none) -> IC: EEPROM 64KBIT I2C [AT24C64D-SSHM-T] [8-SOIC]
Changed lines of the file:
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@@
 					(size 1.27 1.27)
 				)
+				(hide yes)
 			)
 		)
@@
 			)
 		)
-		(property "MPN" "BSE-040-01-X-D-A"
+		(property "MPN" "BSE-040-01-F-D-A-TR"
 			(at 91.44 71.12 0)
 			(effects
@@
 		)
 		(property "OEPSPN" "OEPS070100"
+			(at 91.44 71.12 0)
+			(effects
+				(font
+					(size 1.27 1.27)
+				)
+				(hide yes)
+			)
+		)
+		(property "OEPS DESC" "CONNECTOR:   CONN RCPT 80POS SMD GOLD   [BSE-040-01-F-D-A-TR] [SMD]"
 			(at 91.44 71.12 0)
 			(effects
@@
 					(size 1.27 1.27)
 				)
+				(hide yes)
 			)
 		)
@@
 			)
 		)
-		(property "MPN" "BSE-040-01-X-D-A"
+		(property "MPN" "BSE-040-01-F-D-A-TR"
 			(at 201.93 71.12 0)
 			(effects
@@
 		)
 		(property "OEPSPN" "OEPS070100"
+			(at 201.93 71.12 0)
+			(effects
+				(font
+					(size 1.27 1.27)
+				)
+				(hide yes)
+			)
+		)
+		(property "OEPS DESC" "CONNECTOR:   CONN RCPT 80POS SMD GOLD   [BSE-040-01-F-D-A-TR] [SMD]"
 			(at 201.93 71.12 0)
 			(effects
@@
 					(size 1.27 1.27)
 				)
+				(hide yes)
 			)
 		)
@@
 		)
 		(property "OEPSPN" "OEPS020027"
+			(at 49.53 153.67 0)
+			(effects
+				(font
+					(size 1.27 1.27)
+				)
+				(hide yes)
+			)
+		)
+		(property "OEPS DESC" "RESISTOR:   SMD 0402 1kΩ ±1% 0.063W   [CRCW04021K00FKED] [SMD]"
 			(at 49.53 153.67 0)
 			(effects
@@
 					(size 1.27 1.27)
 				)
+				(hide yes)
 			)
 		)
@@
 		)
 		(property "OEPSPN" "OEPS020027"
+			(at 58.42 153.67 0)
+			(effects
+				(font
+					(size 1.27 1.27)
+				)
+				(hide yes)
+			)
+		)
+		(property "OEPS DESC" "RESISTOR:   SMD 0402 1kΩ ±1% 0.063W   [CRCW04021K00FKED] [SMD]"
 			(at 58.42 153.67 0)
 			(effects
@@
 					(size 1.27 1.27)
 				)
+				(hide yes)
 			)
 		)
@@
 		)
 		(property "OEPSPN" "OEPS020027"
+			(at 67.31 153.67 0)
+			(effects
+				(font
+					(size 1.27 1.27)
+				)
+				(hide yes)
+			)
+		)
+		(property "OEPS DESC" "RESISTOR:   SMD 0402 1kΩ ±1% 0.063W   [CRCW04021K00FKED] [SMD]"
 			(at 67.31 153.67 0)
 			(effects
@@
 				)
 				(justify left)
+				(hide yes)
 			)
 		)
@@
 		)
 		(property "OEPSPN" "OEPS080150"
+			(at 96.52 163.83 0)
+			(effects
+				(font
+					(size 1.27 1.27)
+				)
+				(hide yes)
+			)
+		)
+		(property "OEPS DESC" "IC:   EEPROM 64KBIT I2C   [AT24C64D-SSHM-T] [8-SOIC]"
 			(at 96.52 163.83 0)
 			(effects
@@
 				)
 				(justify right)
+				(hide yes)
 			)
 		)
@@
 			(at 100.33 149.86 0)
 			(effects
+				(font
+					(size 1.27 1.27)
+				)
+				(hide yes)
+			)
+		)
+		(property "OEPS DESC" "CAPACITOR:   SMD CER 0402 100nF 25V ±10% X7R (OEPS H02 001)   [C1005X7R1E104K050BB] [SMD]"
+			(at 100.33 149.86 0)
+			(effects
